File: motor_bldc_esc_V1.kicad_sch (KiCad schematic)
At the start: 1 part, among them J2 Conn_01x03_Socket

Commit message: update pcb (no errors with XRC)
Other:
- sheet PowerStage ports: added none; removed PCB_temp
- sheet mcu ports: added none; removed PCB_temp
Changed lines of the file:
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@@
-	(wire
-		(pts
-			(xy 100.33 110.49) (xy 97.79 110.49)
-		)
-		(stroke
-			(width 0)
-			(type default)
-		)
-	)
 	(wire
 		(pts
@@
 	(wire
 		(pts
-			(xy 212.09 110.49) (xy 207.01 110.49)
-		)
-		(stroke
-			(width 0)
-			(type default)
-		)
-	)
-	(wire
-		(pts
 			(xy 210.82 85.09) (xy 210.82 86.36)
 		)
@@
 	(wire
 		(pts
-			(xy 212.09 118.11) (xy 212.09 110.49)
-		)
-		(stroke
-			(width 0)
-			(type default)
-		)
-	)
-	(wire
-		(pts
 			(xy 95.25 120.65) (xy 214.63 120.65)
 		)
@@
 	(wire
 		(pts
-			(xy 97.79 110.49) (xy 97.79 118.11)
-		)
-		(stroke
-			(width 0)
-			(type default)
-		)
-	)
-	(wire
-		(pts
 			(xy 207.01 104.14) (xy 217.17 104.14)
 		)
@@
 		(pts
 			(xy 93.98 121.92) (xy 93.98 102.87)
-		)
-		(stroke
-			(width 0)
-			(type default)
-		)
-	)
-	(wire
-		(pts
-			(xy 97.79 118.11) (xy 212.09 118.11)
 		)
 		(stroke
@@
 			)
 		)
-		(pin "PCB_temp" output
-			(at 207.01 110.49 0)
-			(effects
-				(font
-					(size 1.27 1.27)
-				)
-				(justify right)
-			)
-		)
 		(instances
 			(project "motor_bldc_esc_V1"
@@
 			(effects
 				(font
-					(size 1.27 1.27)
-				)
-				(justify left)
-			)
-		)
-		(pin "PCB_temp" input
-			(at 100.33 110.49 180)
-			(effects
-				(font

Commit message: finished design of PCB
Parts:
- added H1, H2, H3, H4: MountingHole, MountingHole:MountingHole_3.2mm_M3, symbol Mechanical:MountingHole
