File: power.kicad_sch (KiCad schematic)
At the start: 37 parts, among them J5 Conn_01x02_Socket, U4 TLV75533PDBVR, U5 TI LM5164DDAR

Commit message: edit symbols because of DRC errors (DRV and LM5164)
Parts:
- L1: LCSC Part # C42380259 -> C206289
- U5: footprint Package_SO:HSOP-8-1EP_3.9x4.9mm_P1.27mm_EP2.41x3.1mm_ThermalVias -> Custom:LM5164DDAR
Changed lines of the file:
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@@
 			)
 		)
-		(property "Footprint" "Package_SO:HSOP-8-1EP_3.9x4.9mm_P1.27mm_EP2.41x3.1mm_ThermalVias"
+		(property "Footprint" "Custom:LM5164DDAR"
 			(at 106.68 104.14 0)
 			(hide yes)
@@
 			)
 		)
-		(property "Datasheet" "https://www.lcsc.com/product-detail/C42380259.html?s_z=n_q_t_inductor&spm=wm.fly.bg.3.xh___wm.ssy.tc.0.tz&lcsc_vid=QlcIUVJQQgMNAlZXQ1UMBVAFFVlZVwVfFVlYV1dXE1ExVlNeQlFaX1BWQ1BcUzsOAxUeFF5JWBYZEEoKFBINSQcJGk4%3D"
+		(property "Datasheet" "https://jlcpcb.com/partdetail/SunltechTech-SLW8040S390MST/C206289"
 			(at 148.59 90.17 0)
 			(hide yes)
@@
 			)
 		)
-		(property "Description" "FIXED IND 39uH 1.9A SMD,8x8mm"
+		(property "Description" "1.7A 1.95A 139mΩ 39uH Magnetic Shielded Inductor ±20% SMD,8x8mm Power Inductors ROHS"
 			(at 148.59 90.17 0)
 			(hide yes)
@@
 			)
 		)
-		(property "LCSC Part #" "C42380259"
+		(property "LCSC Part #" "C206289"
 			(at 148.59 90.17 90)
 			(hide yes)

Commit message: update pcb (no errors with XRC)
Parts:
- C31: footprint Custom:100ZLJ330M12.5X35 -> MyLib:100ZLJ330M12.5X35; now in the parts list
- C32: footprint Custom:100ZLJ330M12.5X35 -> MyLib:100ZLJ330M12.5X35
- U5: footprint Custom:LM5164DDAR -> MyLib:LM5164DDAR
Changed lines of the file:
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@@
 			)
 		)
-		(property "Footprint" "Custom:LM5164DDAR"
+		(property "Footprint" "MyLib:LM5164DDAR"
 			(at 106.68 104.14 0)
 			(hide yes)
@@
 		(body_style 1)
 		(exclude_from_sim no)
-		(in_bom no)
+		(in_bom yes)
 		(on_board yes)
 		(in_pos_files yes)
@@
 			)
 		)
-		(property "Footprint" "Custom:100ZLJ330M12.5X35"
+		(property "Footprint" "MyLib:100ZLJ330M12.5X35"
 			(at 59.3852 46.99 0)
 			(hide yes)
@@
 						(name "HighCurrent")
 						(dnp no)
-						(in_bom yes)
 					)
 					(variant
 						(name "HighCurrent2")
 						(dnp no)
-						(in_bom yes)
 					)
 					(variant
 						(name "LowCurrent")
-						(in_bom yes)
 					)
 					(variant
 						(name "LowCurrent1")
 						(dnp no)
-						(in_bom yes)
 					)
 				)
@@
 			)
 		)
-		(property "Footprint" "Custom:100ZLJ330M12.5X35"
+		(property "Footprint" "MyLib:100ZLJ330M12.5X35"
 			(at 72.0852 46.99 0)
 			(hide yes)

Commit message: changes MCU because of stock
Parts:
- D7: value LED_Status -> LED_5V
- D8: value LED_Status -> LED_3V3
Changed lines of the file:
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@@
 			)
 		)
-		(property "Value" "LED_Status"
+		(property "Value" "LED_5V"
 			(at 215.9 47.3074 90)
 			(show_name no)
@@
 			)
 		)
-		(property "Value" "LED_Status"
+		(property "Value" "LED_3V3"
 			(at 199.39 47.3074 90)
 			(show_name no)
